Commit message: fix: fix fira action json

File: umaru/urdf/umaru.urdf (robot description, URDF)
Before this commit: robot UMARU, 26 links, 25 joints
Links:
- link body: geometry collision mesh filename=file://meshes/teen_size/Body.stl scale=0.001 0.001 0.001; visual mesh filename=file://meshes/teen_size/Body.stl scale=0.001 0.001 0.001
- link head: geometry collision mesh filename=file://meshes/teen_size/Head.stl scale=0.001 0.001 0.001; visual mesh filename=file://meshes/teen_size/Head.stl scale=0.001 0.001 0.001
- link left_buttock: geometry collision mesh filename=file://meshes/teen_size/Buttock.stl scale=0.001 0.001 0.001; visual mesh filename=file://meshes/teen_size/Buttock.stl scale=0.001 0.001 0.001
- link left_calf: geometry collision mesh filename=file://meshes/teen_size/Calf.stl scale=0.001 0.001 0.001; visual mesh filename=file://meshes/teen_size/Calf.stl scale=0.001 0.001 0.001
- link left_foot: geometry collision mesh filename=file://meshes/teen_size/Left_Foot.stl scale=0.001 0.001 0.001; visual mesh filename=file://meshes/teen_size/Left_Foot.stl scale=0.001 0.001 0.001
- link left_forearm: geometry collision mesh filename=file://meshes/teen_size/Forearm.stl scale=0.001 0.001 0.001; visual mesh filename=file://meshes/teen_size/Forearm.stl scale=0.001 0.001 0.001
- link left_groin: geometry collision mesh filename=file://meshes/teen_size/Groin.stl scale=0.001 0.001 0.001; visual mesh filename=file://meshes/teen_size/Groin.stl scale=0.001 0.001 0.001
- link left_heel: geometry collision mesh filename=file://meshes/teen_size/Heel.stl scale=0.001 0.001 0.001; visual mesh filename=file://meshes/teen_size/Heel.stl scale=0.001 0.001 0.001
- link left_shoulder: geometry collision mesh filename=file://meshes/teen_size/Shoulder.stl scale=0.001 0.001 0.001; visual mesh filename=file://meshes/teen_size/Shoulder.stl scale=0.001 0.001 0.001
- link left_thigh: geometry collision mesh filename=file://meshes/teen_size/Thigh.stl scale=0.001 0.001 0.001; visual mesh filename=file://meshes/teen_size/Thigh.stl scale=0.001 0.001 0.001
- link left_upper_arm: geometry collision mesh filename=file://meshes/teen_size/Upper_Arm.stl scale=0.001 0.001 0.001; visual mesh filename=file://meshes/teen_size/Upper_Arm.stl scale=0.001 0.001 0.001
- link neck: geometry collision mesh filename=file://meshes/teen_size/Neck.stl scale=0.001 0.001 0.001; visual mesh filename=file://meshes/teen_size/Neck.stl scale=0.001 0.001 0.001
- link right_buttock: geometry collision mesh filename=file://meshes/teen_size/Buttock.stl scale=0.001 0.001 0.001; visual mesh filename=file://meshes/teen_size/Buttock.stl scale=0.001 0.001 0.001
- link right_calf: geometry collision mesh filename=file://meshes/teen_size/Calf.stl scale=0.001 0.001 0.001; visual mesh filename=file://meshes/teen_size/Calf.stl scale=0.001 0.001 0.001
- link right_foot: geometry collision mesh filename=file://meshes/teen_size/Right_Foot.stl scale=0.001 0.001 0.001; visual mesh filename=file://meshes/teen_size/Right_Foot.stl scale=0.001 0.001 0.001
- link right_forearm: geometry collision mesh filename=file://meshes/teen_size/Forearm.stl scale=0.001 0.001 0.001; visual mesh filename=file://meshes/teen_size/Forearm.stl scale=0.001 0.001 0.001
- link right_groin: geometry collision mesh filename=file://meshes/teen_size/Groin.stl scale=0.001 0.001 0.001; visual mesh filename=file://meshes/teen_size/Groin.stl scale=0.001 0.001 0.001
- link right_heel: geometry collision mesh filename=file://meshes/teen_size/Heel.stl scale=0.001 0.001 0.001; visual mesh filename=file://meshes/teen_size/Heel.stl scale=0.001 0.001 0.001
- link right_shoulder: geometry collision mesh filename=file://meshes/teen_size/Shoulder.stl scale=0.001 0.001 0.001; visual mesh filename=file://meshes/teen_size/Shoulder.stl scale=0.001 0.001 0.001
- link right_thigh: geometry collision mesh filename=file://meshes/teen_size/Thigh.stl scale=0.001 0.001 0.001; visual mesh filename=file://meshes/teen_size/Thigh.stl scale=0.001 0.001 0.001
- link right_upper_arm: geometry collision mesh filename=file://meshes/teen_size/Upper_Arm.stl scale=0.001 0.001 0.001; visual mesh filename=file://meshes/teen_size/Upper_Arm.stl scale=0.001 0.001 0.001
Joints:
- joint camera_joint: origin xyz=0.0 0.020000000000000004 0.04000000000000001 rpy=-1.5707963267948966 3.141592653589793 0 -> xyz=0.0 0.020000000000000004 0.04000000000000001 rpy=-1.5707963267948966 0 0
